Commit message: arduin test motor surme devresi ve kodları olusturuldu. Bu uygulamada sadece deneme amaclı olarak doğrudan serial üzerinden ROS'A baglanarak 0-255 arası data alıp bunları l298 motor surucusu ile calıstırdım. Gayet basarılı

File: jackal_car_dagu/jackal_car_description/urdf/jackal_car.xacro (robot description, xacro)
@@ -60,5 +60,5 @@
  	 <inertial>
 	  <origin xyz="0 0 0" rpy="0 0 0" />
-	   <mass value="0.555250122552161" />
+	   <!--<mass value="0.555250122552161" />
 	    <inertia
 		ixx="0.0018554608262"
@@ -68,4 +68,13 @@
 		iyz="0.0"
 		izz="0.0023135421773"/>
+	 </inertial>-->
+	<mass value="1.755250122552161" />
+	    <inertia
+		ixx="0.01479"
+		ixy="0.0"
+		ixz="0.0"
+		iyy="0.02703"
+		iyz="0.0"
+		izz="0.03774"/>
 	 </inertial>
 	 <visual>

Commit message: I've implemented of joystick board and utility soft.

File: jackal_car_dagu/jackal_car_description/urdf/jackal_car.xacro (robot description, xacro)
@@ -38,7 +38,7 @@
 	<xacro:property name="rpy_l_2" value="1.70172090315557 0.839815899464149 -3.04386814481467"/>-->
 	<xacro:property name="xyz_l_1" value="0 0.155934743 -0.0334984052243152"/>
-		<xacro:property name="rpy_l_1" value="-1.480796105 0.160636578101035 -3.12741615571841"/>
+	<xacro:property name="rpy_l_1" value="-1.480796105 0.160636578101035 -3.12741615571841"/>
 	<xacro:property name="xyz_l_0" value="-0.146 0.155934743 -0.0346340445573322"/>
-		<xacro:property name="rpy_l_0" value="1.293379552 1.24503993158855 -0.261989767251398"/>
+	<xacro:property name="rpy_l_0" value="1.293379552 1.24503993158855 -0.261989767251398"/>
 	<xacro:property name="xyz_l_2" value="0.146 0.155934743 -0.0332465540892745"/>
 	<xacro:property name="rpy_l_2" value="-1.438279097 0.839815899464149 -3.04386814481467"/>
@@ -60,5 +60,5 @@
  	 <inertial>
 	  <origin xyz="0 0 0" rpy="0 0 0" />
-	   <!--<mass value="0.555250122552161" />
+	<!--   <mass value="0.555250122552161" />
 	    <inertia
 		ixx="0.0018554608262"
@@ -69,12 +69,12 @@
 		izz="0.0023135421773"/>
 	 </inertial>-->
-	<mass value="1.755250122552161" />
+	<mass value="0.0255250122552161" />
 	    <inertia
-		ixx="0.01479"
+		ixx="0.001479"
 		ixy="0.0"
 		ixz="0.0"
-		iyy="0.02703"
+		iyy="0.0002703"
 		iyz="0.0"
-		izz="0.03774"/>
+		izz="0.003774"/>
 	 </inertial>
 	 <visual>
@@ -123,5 +123,5 @@
 	 </collision>
   	</link>
-	<link name="h_realsense_0">
+	<!-- --><link name="h_realsense_0">
     	 <inertial>
          <origin xyz="0 0 0" rpy="0 0 0" />
@@ -154,5 +154,5 @@
 	    <axis   xyz="1 0 0" />
 	</joint>
-	<link name="laser">
+	 <link name="laser">
 	<inertial>
 	        <mass value="1.1" />
